File: 03 bottom_plate/therick48_bottom_plate.kicad_pcb (KiCad board)
At the start: 2 copper layers, 228 x 76 mm, 65 parts, among them U1 HOLE, U10 HOLE, U11 HOLE, U12 HOLE, U13 HOLE, U14 HOLE, U15 HOLE, U16 HOLE, U17 HOLE, U18 HOLE, U19 HOLE, U2 HOLE, U20 HOLE, U21 HOLE, U22 HOLE, U23 HOLE, U24 HOLE, U25 HOLE, U26 HOLE, U27 HOLE, U28 HOLE, U29 HOLE, U3 HOLE, U30 HOLE, U31 HOLE, U32 HOLE, U33 HOLE, U34 HOLE, U35 HOLE, U36 HOLE, U37 HOLE, U38 HOLE, U39 HOLE, U4 HOLE, U40 HOLE, U41 HOLE, U42 HOLE, U43 HOLE, U44 HOLE, U45 HOLE, U46 HOLE, U47 HOLE, U48 HOLE, U49 HOLE, U5 HOLE, U6 HOLE, U65 HOLE, U7 HOLE, U8 HOLE, U9 HOLE

Commit message: Gerber
Other:
- board text added: "github.com/dierickdie"
Changed lines of the file:
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@@
   (general
     (thickness 1.6)
-    (drawings 20)
+    (drawings 21)
     (tracks 0)
     (zones 0)
@@
     (pad 1 thru_hole circle (at 0 0) (size 3.5 3.5) (drill 2.2) (layers *.Cu *.Mask))
   )
-  (gr_text "therick48 Rev 1.1" (at 48.639872 72.959808 90) (layer F.SilkS)
+  (gr_text github.com/dierickdie (at 122.359678 37.619901) (layer F.SilkS)
+    (effects (font (size 1.5 1.5) (thickness 0.2)))
+  )
+  (gr_text "therick48 Rev 1.1" (at 160.359578 37.619901) (layer F.SilkS)
     (effects (font (size 1.5 1.5) (thickness 0.2)))
   )
@@
   (gr_arc (start 50.16 107.16) (end 46.36 107.16) (angle -90) (layer Edge.Cuts) (width 0.15))
   (gr_arc (start 50.16 38.76) (end 50.16 34.96) (angle -90) (layer Edge.Cuts) (width 0.15))
-  (gr_text JLCJLCJLCJLC (at 48.64 106.4 90) (layer F.SilkS)
-    (effects (font (size 1 1) (thickness 0.15)) (justify left))
+  (gr_text JLCJLCJLCJLC (at 49.39987 82.459783 90) (layer F.SilkS)
+    (effects (font (size 1 1) (thickness 0.15)))
   )
   (gr_line (start 217.4875 89.69375) (end 217.4875 94.45625) (layer Dwgs.User) (width 0.15))
